File: eda/where_is_my_ion.kicad_pcb (KiCad board)
At the start: 4 copper layers, 75 x 150 mm, 158 parts, among them J1 USB_C_Receptacle_USB2.0_16P, Q1 L8050QLT1G, Q2 L8050QLT1G, SW1 SW_MCU_RESET, SW2 FORCE_REFRESH, SW3 NEXT_TRAIN, SW4 SW_BOOT_SEL, U1 CP2102N-Axx-xQFN28, U2 TLC59116IPWR, U3 TLC59116IPWR, U4 TLC59116IPWR, U5 TLC59116IPWR, U6 ESP32-C3-WROOM-02, U7 TLC59116IPWR, U8 AP2112K-3.3

Commit message: routing is hard
Parts:
- removed the C11 at (162.5, 121.1)
- removed the C17 at (65.1, 118.4)
- C15: value 1 uF/50V (NC) -> 10uF; footprint Capacitor_SMD:C_0805_2012Metric -> Capacitor_Tantalum_SMD:CP_EIA-3528-15_AVX-H
- moved C1 57.7 mm to (167.0, 154.4)
- moved R3 47.7 mm to (175.8, 155.9)
- moved C6 47.5 mm to (161.9, 159.2), turned to 90 degrees
- moved R2 47.5 mm to (173.2, 155.9)
- moved C15 47.1 mm to (62.9, 130.4)
- moved Q1 47.1 mm to (63.3, 135.2)
- moved R11 47.1 mm to (67.9, 137.2)
- moved R9 47.1 mm to (67.9, 139.6)
- moved SW4 47.1 mm to (59.0, 131.7)
- moved Q2 47.1 mm to (63.0, 141.4)
- moved SW1 47.1 mm to (59.0, 140.3)
- moved R6 46.8 mm to (161.4, 164.0)
- moved U1 46.6 mm to (167.1, 161.7)
- moved R5 45.2 mm to (159.8, 159.3), turned to 90 degrees
- moved R1 42.8 mm to (161.4, 162.1), turned to 0 degrees
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- renumbered C12 to C11, C13 to C12, C14 to C13, C16 to C14, C18 to C16, C19 to C17, C20 to C18, C21 to C19
Connections:
- net Net-(D83-A2) renamed /USB_D-
- net Net-(D84-A2) renamed /USB_D+
- C15 pad 1: GND -> +3V3
- C15 pad 2: /CHIP_PU -> GND
Routing:
- net /USB_D+: track 0.00 -> 39.3 mm
- net GND: track 0.00 -> 39.0 mm
- net /USB_D-: track 0.00 -> 34.6 mm
- net +3V3: track 0.00 -> 30.4 mm
- net /VBUS: track 0.00 -> 20.6 mm
- net /IO18: track 0.00 -> 19.7 mm, vias 0 -> 2
- net +5V: track 0.00 -> 19.6 mm
- net /U0RXD: track 0.00 -> 18.8 mm
- net /IO5_SDA: track 0.00 -> 18.3 mm
- net /USB_DP: track 0.00 -> 18.2 mm
- net /IO19: track 0.00 -> 16.7 mm, vias 0 -> 2
- net /U0TXD: track 0.00 -> 15.8 mm, vias 0 -> 2
- net /IO8: track 0.00 -> 14.6 mm
- net /IO6_SCL: track 0.00 -> 13.2 mm
- net /IO4_~{RESET}: track 0.00 -> 12.9 mm, vias 0 -> 3
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- added copper zone on In2.Cu, net +3V3
- added copper zone on In1.Cu, net GND

Commit message: commit
Parts:
- C10, C14, C15, C7, C8, C9, D25, D26, D27, D28, D29, D30, D31, D32, D41, D42, D43, D44, D45, D46, D47, D48, D56, D57, D58, D59, D60, D61, D62, D63, D64, D65, D66, D67, D68, D70, D71, D76, D77, D78, D80, Q1, Q2, R11, R12, R7, R9, SW1, SW4, U2, U5: moved to B.Cu
- D69, D79: value LED_INTER_WHITE -> LED_STN_BLUE; moved to B.Cu
- moved C9 156.6 mm to (174.2, 73.8), turned to 180 degrees
- moved D30 151.3 mm to (173.5, 144.2)
- moved SW4 150.2 mm to (204.9, 167.3), turned to -90 degrees
- moved D28 149.7 mm to (173.0, 133.8)
- moved D32 148.6 mm to (168.0, 154.5)
- moved D26 148.0 mm to (170.5, 126.0)
- moved SW1 147.1 mm to (204.9, 158.8), turned to -90 degrees
- moved D29 146.1 mm to (173.5, 138.8)
- moved D31 144.4 mm to (171.2, 149.2)
- moved D27 144.4 mm to (170.8, 130.0)
- moved R12 142.4 mm to (174.6, 85.8), turned to 180 degrees
- moved D25 142.0 mm to (166.7, 118.8)
- moved D48 127.3 mm to (165.5, 115.2), turned to 180 degrees
- moved Q2 127.2 mm to (183.5, 182.0), turned to 0 degrees
- moved U5 124.1 mm to (171.2, 79.8), turned to 90 degrees
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Routing:
- net /IO6_SCL: track 13.2 -> 129.1 mm, vias 0 -> 4
- net /IO5_SDA: track 18.3 -> 130.7 mm, vias 0 -> 4
- net /IO4_~{RESET}: track 12.9 -> 117.3 mm, vias 3 -> 7
- net GND: track 39.0 -> 105.8 mm, vias 0 -> 13
- net /STN_BORDEN: track 0.00 -> 47.8 mm
- net /INTER_kmrkt_borden_2: track 0.00 -> 45.4 mm
- net /INTER_borden_mill_1: track 0.00 -> 44.6 mm
- net /INTER_kmrkt_borden_1: track 0.00 -> 44.4 mm
- net /STN_MILL: track 0.00 -> 44.4 mm, vias 0 -> 2
- net /INTER_wloosq_lwp: track 0.00 -> 39.7 mm
- net /INTER_borden_mill_2: track 0.00 -> 39.6 mm
- net /STN_ALLEN: track 0.00 -> 39.2 mm, vias 0 -> 1
- net /STN_KCHNR_MRKT: track 0.00 -> 37.5 mm
- net /STN_WILLIS_WAY: track 0.00 -> 34.3 mm, vias 0 -> 1
- net /STN_REV_WLOO_SQ: track 0.00 -> 33.3 mm
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
Commit message: changes
Parts:
- C10: moved to F.Cu
- D45: value LED_INTER_WHITE -> LED_STN_BLUE
- D46: value LED_STN_BLUE -> LED_INTER_WHITE
- U3: moved to B.Cu
- moved TP1 173.7 mm to (198.4, 100.7)
- moved TP2 173.7 mm to (198.2, 83.8)
- moved TP3 173.7 mm to (198.4, 104.7)
- moved TP4 173.7 mm to (198.2, 87.8)
- moved TP5 173.7 mm to (198.4, 108.8)
- moved TP6 173.7 mm to (198.2, 91.9)
- moved TP7 173.7 mm to (198.4, 112.8)
- moved TP8 173.7 mm to (198.2, 96.0)
- moved TP9 173.7 mm to (198.4, 116.8)
- moved D81 92.6 mm to (152.3, 178.2)
- moved R21 92.6 mm to (149.1, 178.1)
- moved R10 89.4 mm to (113.7, 83.4)
- moved D49 83.6 mm to (104.7, 68.9), turned to -90 degrees
- moved C4 61.3 mm to (82.0, 112.8)
- moved U3 54.2 mm to (139.7, 134.9), turned to 90 degrees
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Connections:
- D44 pad 1: /INTER_borden_kmrkt_2 -> /INTER_borden_kmrkt_1
- D45 pad 1: /INTER_borden_kmrkt_1 -> /STN_REV_BORDEN
- D46 pad 1: /STN_REV_BORDEN -> /INTER_mill_borden_2
- U5 pad 11: /INTER_borden_kmrkt_2 -> /INTER_borden_kmrkt_1
- U5 pad 7: /INTER_mill_borden_1 -> /INTER_mill_borden_2
- U5 pad 8: /STN_REV_BORDEN -> /INTER_mill_borden_1
- U5 pad 9: /INTER_borden_kmrkt_1 -> /STN_REV_BORDEN
Routing:
- net /STN_REV_MILL: track 0.00 -> 35.9 mm
- net /STN_REV_BORDEN: track 0.00 -> 35.4 mm
- net /INTER_mill_borden_1: track 0.00 -> 34.0 mm
- net /INTER_mill_borden_2: track 0.00 -> 32.7 mm
- net /INTER_borden_kmrkt_1: track 0.00 -> 30.7 mm
- net /STN_REV_KTCHNR_MRKT: track 0.00 -> 25.7 mm
- net /STN_REV_FREDERICK: track 0.00 -> 22.1 mm
- net /STN_REV_CITY_HALL: track 0.00 -> 18.3 mm
- net /INTER_wloosq_lwp: track 39.7 -> 50.8 mm
- net /STN_REV_WLOO_SQ: track 33.3 -> 42.2 mm
- net /STN_REV_ALLEN: track 29.5 -> 36.0 mm
- net GND: track 105.8 -> 110.3 mm, vias 13 -> 22
- net /INTER_grh_allen_1: track 26.8 -> 30.3 mm
- net Net-(U4-REXT): track 0.00 -> 2.93 mm
- net /STN_REV_GRH: track 23.5 -> 24.6 mm
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
Commit message: stuff
Parts:
- R8: moved to B.Cu
- moved C5 83.2 mm to (142.2, 138.0), turned to 180 degrees
- moved R8 70.7 mm to (146.2, 138.7), turned to -90 degrees
- moved C4 64.5 mm to (142.5, 135.0), turned to 180 degrees
- moved D15 0.51 mm to (109.0, 124.2), turned to 180 degrees
- moved D11 0.25 mm to (105.0, 144.2), turned to 180 degrees
- moved D12 0.25 mm to (104.8, 138.8), turned to 180 degrees
- moved D16 0.20 mm to (110.8, 120.0), turned to 180 degrees
- moved D10 0.15 mm to (108.2, 149.0), turned to 180 degrees
- moved D14 0.15 mm to (108.0, 129.8), turned to 180 degrees
- moved D9 0.10 mm to (111.2, 153.5), turned to 180 degrees
- turned D13 to 180 degrees
Routing:
- net /INTER_fairway_block_1: track 0.00 -> 44.5 mm, vias 0 -> 4
- net /STN_REV_FAIRWAY: track 0.00 -> 43.6 mm, vias 0 -> 2
- net /INTER_fairway_block_2: track 0.00 -> 41.5 mm
- net /STN_BLOCK_LINE: track 0.00 -> 39.1 mm, vias 0 -> 1
- net /INTER_fairway_block_3: track 0.00 -> 38.6 mm
- net /INTER_block_fairway_1: track 0.00 -> 38.0 mm, vias 0 -> 1
- net /INTER_mill_block_3: track 0.00 -> 37.3 mm, vias 0 -> 1
- net /INTER_mill_block_1: track 0.00 -> 37.0 mm, vias 0 -> 1
- net /INTER_mill_block_2: track 0.00 -> 36.3 mm, vias 0 -> 1
- net /INTER_block_fairway_2: track 0.00 -> 36.1 mm, vias 0 -> 1
- net /INTER_block_mill_1: track 0.00 -> 35.9 mm, vias 0 -> 4
- net /STN_REV_BLOCK_LINE: track 0.00 -> 35.8 mm
- net /IO4_~{RESET}: track 117.3 -> 152.6 mm, vias 7 -> 10
- net /INTER_block_mill_2: track 0.00 -> 34.0 mm, vias 0 -> 2
- net /INTER_block_fairway_3: track 0.00 -> 32.4 mm, vias 0 -> 1
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
Commit message: almost done; might have to redo driver2
Parts:
- removed TP6, TP7, TP8, TP9: TestPoint, TestPoint:TestPoint_Pad_D2.0mm
- TP1, TP2, TP3, TP4, TP5: moved to B.Cu
- moved D81 161.3 mm to (139.8, 17.3), turned to 180 degrees
- moved R21 158.8 mm to (139.9, 19.6), turned to 180 degrees
- moved TP5 142.9 mm to (70.4, 45.2)
- moved TP3 137.6 mm to (70.2, 54.6)
- moved TP1 133.6 mm to (69.9, 64.0)
- moved TP4 133.6 mm to (70.2, 49.7)
- moved TP2 130.3 mm to (70.2, 59.2)
- moved SW4 110.8 mm to (106.2, 117.0)
- moved SW1 101.9 mm to (112.0, 117.0)
- moved Q2 89.2 mm to (106.7, 136.5)
- moved Q1 74.8 mm to (106.7, 131.4)
- moved SW2 67.2 mm to (155.1, 141.5), turned to 180 degrees
- moved SW3 66.7 mm to (155.1, 145.8), turned to 180 degrees
- moved R11 47.7 mm to (126.8, 163.3), turned to 180 degrees
- moved R9 45.5 mm to (126.8, 160.7), turned to 180 degrees
Connections:
- TP2 pad 1: /IO2 -> +3V3
- TP3 pad 1: +3V3 -> /IO5_SDA
- TP4 pad 1: /IO3 -> /IO6_SCL
- TP5 pad 1: /IO5_SDA -> /IO4_~{RESET}
Routing:
- net /~{RTS}: track 0.00 -> 87.5 mm, vias 0 -> 2
- net /IO9: track 0.57 -> 83.8 mm, vias 0 -> 1
- net /CHIP_PU: track 9.90 -> 92.7 mm, vias 2 -> 6
- net /~{DTR}: track 0.00 -> 79.2 mm, vias 0 -> 3
- net /IO6_SCL: track 148.5 -> 204.0 mm, vias 5 -> 8
- net /IO5_SDA: track 152.8 -> 204.9 mm, vias 5 -> 7
- net /IO4_~{RESET}: track 152.6 -> 203.1 mm, vias 10 -> 12
- net Net-(Q1-B): track 0.00 -> 39.1 mm
- net Net-(Q2-B): track 0.00 -> 35.9 mm
- net /IO0_SW: track 0.00 -> 21.0 mm
- net /IO1_SW: track 0.00 -> 18.3 mm, vias 0 -> 2
- net /STN_MILL: track 44.4 -> 58.5 mm
- net GND: track 118.4 -> 114.5 mm, vias 24 -> 25
- net +3V3: track 69.2 -> 66.3 mm, vias 13 -> 14
- net Net-(D81-A): track 0.11 -> 2.31 mm
