File: eda/where_is_my_ion.kicad_pcb (KiCad board)
At the start: 4 copper layers, 75 x 150 mm, 152 parts, among them J1 USB_C_Receptacle_USB2.0_16P, Q1 L8050QLT1G, Q2 L8050QLT1G, SW1 SW_MCU_RESET, SW2 FORCE_REFRESH, SW3 NEXT_TRAIN, SW4 SW_BOOT_SEL, U1 CP2102N-Axx-xQFN28, U2 TLC59116IPWR, U3 TLC59116IPWR, U4 TLC59116IPWR, U5 TLC59116IPWR, U6 ESP32-C3-WROOM-02, U7 TLC59116IPWR, U8 AP2112K-3.3

Commit message: might change
Parts:
- added TP10: TestPoint, TestPoint:TestPoint_Pad_D2.0mm, B.Cu at (128.2, 153.8)
- added TP6: TestPoint, TestPoint:TestPoint_Pad_D2.0mm, B.Cu at (133.0, 153.8)
- added TP7: TestPoint, TestPoint:TestPoint_Pad_D2.0mm, B.Cu at (138.0, 153.8)
- added TP8: TestPoint, TestPoint:TestPoint_Pad_D2.0mm, B.Cu at (142.5, 153.8)
- added TP9: TestPoint, TestPoint:TestPoint_Pad_D2.0mm, B.Cu at (147.0, 153.5)
- moved TP1 107.9 mm to (174.2, 36.5)
- moved TP2 107.7 mm to (174.3, 31.7)
- moved TP3 104.9 mm to (174.2, 41.5)
- moved TP4 104.1 mm to (174.2, 46.0)
- moved TP5 104.0 mm to (174.2, 51.0)
Routing:
- net /IO5_SDA: track 204.9 -> 282.3 mm, vias 7 -> 11
- net /IO4_~{RESET}: track 203.1 -> 256.1 mm
- net /IO6_SCL: track 204.0 -> 249.0 mm
- net /IO9: track 83.8 -> 117.8 mm, vias 1 -> 3
- net /IO0_SW: track 21.0 -> 50.4 mm, vias 0 -> 1
- net /U0RXD: track 18.8 -> 46.0 mm, vias 0 -> 1
- net /IO1_SW: track 18.3 -> 43.6 mm, vias 2 -> 3
- net /U0TXD: track 15.8 -> 37.5 mm, vias 2 -> 4
- net /STN_MILL: track 58.5 -> 51.5 mm
- net GND: track 114.5 -> 115.1 mm

Commit message: side by side layout
Parts:
- removed D54: LED_INTER_WHITE, LED_SMD:LED_0603_1608Metric
- D25, D26, D27, D28, D29, D30, D31, D32, D41, D42, D43, D44, D45, D46, D47, D48, D56, D57, D58, D59, D60, D61, D62, D63, D64, D65, D66, D67, D68, D69, D70, D71, D76, D77, D78, D79, D80: moved to F.Cu
- moved U3 296.4 mm to (-156.7, 127.7)
- moved R8 289.8 mm to (-139.7, 91.4)
- moved C5 286.3 mm to (-139.2, 85.4)
- moved C4 284.1 mm to (-136.1, 79.4)
- moved C10 233.6 mm to (-54.9, 30.7)
- moved C14 233.6 mm to (-108.5, -4.34)
- moved C2 233.6 mm to (-71.8, -8.99)
- moved C3 233.6 mm to (-69.0, -9.04)
- moved C7 233.6 mm to (-124.2, 33.9)
- moved C8 233.6 mm to (-121.2, 33.7)
- moved C9 233.6 mm to (-54.8, 27.3)
- moved D49 233.6 mm to (-124.2, 22.3)
- moved R10 233.6 mm to (-115.2, 36.8)
- moved R18 233.6 mm to (-105.9, 0.21)
- moved R7 233.6 mm to (-68.7, -13.3)
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Connections:
- U4 pad 20: /INTER_borden_mill_2 -> /STN_MILL
- U4 pad 21: /STN_MILL -> /LED_IS_FETCHING
- U4 pad 22: /LED_IS_FETCHING -> unconnected-(U4-~{OUT14}-Pad22)
Routing:
- net /IO5_SDA: track 282.3 -> 24.3 mm, vias 11 -> 1
- net /IO4_~{RESET}: track 256.1 -> 15.1 mm, vias 12 -> 4
- net /IO6_SCL: track 249.0 -> 18.4 mm, vias 8 -> 1
- net /IO9: track 117.8 -> 16.3 mm, vias 3 -> 0
- net /CHIP_PU: track 92.7 -> 11.6 mm, vias 6 -> 2
- net GND: track 115.1 -> 37.0 mm, vias 25 -> 7
- net /STN_MILL: track 51.5 -> 0.00 mm, vias 2 -> 0
- net /INTER_wloosq_lwp: track 50.8 -> 0.00 mm
- net /STN_BORDEN: track 47.8 -> 0.00 mm
- net /INTER_kmrkt_borden_2: track 45.4 -> 0.00 mm
- net /INTER_borden_mill_1: track 44.6 -> 0.00 mm
- net /INTER_fairway_block_1: track 44.5 -> 0.00 mm, vias 4 -> 0
- net /INTER_kmrkt_borden_1: track 44.4 -> 0.00 mm
- net /STN_REV_FAIRWAY: track 43.6 -> 0.00 mm, vias 2 -> 0
- net /IO1_SW: track 43.6 -> 0.30 mm, vias 3 -> 0
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Other:
- board size 75 x 150 mm -> 88 x 162.9 mm

Commit message: nearly done
Parts:
- C14, C15, C9: moved to F.Cu
- R10, R18, U4, U7: moved to B.Cu
- moved C15 226.2 mm to (107.5, 52.2), turned to 0 degrees
- moved C14 224.1 mm to (107.5, 55.2), turned to 0 degrees
- moved U3 223.7 mm to (64.9, 158.8), turned to 180 degrees
- moved C5 218.3 mm to (67.7, 155.2), turned to -90 degrees
- moved R8 217.3 mm to (68.8, 152.8), turned to 0 degrees
- moved C4 215.0 mm to (64.9, 155.8), turned to -90 degrees
- moved R18 215.0 mm to (103.0, 51.0), turned to 180 degrees
- moved C7 195.5 mm to (55.4, 111.2), turned to 0 degrees
- moved U4 195.5 mm to (59.6, 105.4), turned to -90 degrees
- moved C8 193.9 mm to (55.4, 113.9), turned to 0 degrees
- moved D49 189.0 mm to (46.0, 104.5), turned to 90 degrees
- moved R10 180.3 mm to (52.8, 102.5), turned to 180 degrees
- moved C9 170.7 mm to (97.0, 105.3)
- moved C10 170.4 mm to (96.9, 108.0)
- moved R12 169.5 mm to (100.6, 107.4), turned to 90 degrees
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Connections:
- U4 pad 16: /INTER_kmrkt_borden_2 -> /STN_BORDEN
- U4 pad 17: /STN_BORDEN -> /INTER_borden_mill_1
- U4 pad 18: /INTER_borden_mill_1 -> /INTER_borden_mill_2
Routing:
- net /IO5_SDA: track 24.3 -> 334.9 mm, vias 1 -> 11
- net /IO4_~{RESET}: track 15.1 -> 311.0 mm, vias 4 -> 11
- net /IO6_SCL: track 18.4 -> 312.6 mm, vias 1 -> 11
- net GND: track 37.0 -> 122.8 mm, vias 7 -> 29
- net /INTER_cstg_nrthf_1: track 0.00 -> 78.0 mm, vias 0 -> 3
- net /INTER_cstg_nrthf_2: track 0.00 -> 66.9 mm, vias 0 -> 3
- net /STN_CONESTOGA: track 0.00 -> 64.7 mm, vias 0 -> 3
- net /IO9: track 16.3 -> 78.7 mm, vias 0 -> 5
- net /STN_NORTHFIELD: track 0.00 -> 56.9 mm, vias 0 -> 1
- net +3V3: track 29.3 -> 84.0 mm, vias 6 -> 15
- net /STN_REV_MILL: track 0.00 -> 52.6 mm, vias 0 -> 3
- net /INTER_nrthf_rnt_1: track 0.00 -> 51.2 mm, vias 0 -> 1
- net /CHIP_PU: track 11.6 -> 60.8 mm, vias 2 -> 5
- net /INTER_wloosq_lwp: track 0.00 -> 47.8 mm, vias 0 -> 1
- net /INTER_mill_borden_1: track 0.00 -> 46.7 mm, vias 0 -> 3
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Other:
- board size 88 x 162.9 mm -> 88 x 163 mm
