File: eda/where_is_my_ion.kicad_sch (KiCad schematic)
At the start: 156 parts, among them J1 USB_C_Receptacle_USB2.0_16P, Q1 L8050QLT1G, Q2 L8050QLT1G, SW1 SW_MCU_RESET, SW2 FORCE_REFRESH, SW3 NEXT_TRAIN, SW4 SW_BOOT_SEL, U1 CP2102N-Axx-xQFN28, U2 TLC59116IPWR, U3 TLC59116IPWR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

Commit message: nearly done
Connections:
- net INTER_kmrkt_borden_2 is gone; now on net STN_BORDEN: U4.16 (~{OUT9})
- net INTER_borden_mill_1: now also U4.17 (~{OUT10}); no longer U4.18 (~{OUT11})
- net INTER_borden_mill_2: now also U4.18 (~{OUT11})
- net STN_BORDEN: no longer U4.17 (~{OUT10})
Changed lines of the file:
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@@
 	(wire
 		(pts
-			(xy 227.33 179.07) (xy 250.19 179.07)
-		)
-		(stroke
-			(width 0)
-			(type default)
-		)
-	)
-	(wire
-		(pts
 			(xy 443.23 63.5) (xy 466.09 63.5)
 		)
@@
 	(wire
 		(pts
+			(xy 227.33 179.07) (xy 250.19 179.07)
+		)
+		(stroke
+			(width 0)
+			(type default)
+		)
+	)
+	(wire
+		(pts
 			(xy 529.59 229.87) (xy 537.21 229.87)
 		)
@@
 	)
 	(label "STN_BORDEN"
-		(at 250.19 171.45 180)
+		(at 250.19 168.91 180)
 		(effects
 			(font
@@
 		)
 	)
+	(label "INTER_borden_mill_2"
+		(at 250.19 173.99 180)
+		(effects
+			(font
+				(size 1.27 1.27)
+			)
+			(justify right bottom)
+		)
+	)
 	(label "IO8"
 		(at 276.86 256.54 0)
@@
 	)
 	(label "INTER_borden_mill_1"
-		(at 250.19 173.99 180)
+		(at 250.19 171.45 180)
 		(effects
 			(font
@@
 		(effects
 			(font
-				(size 1.27 1.27)
-			)
-			(justify right bottom)
-		)
-	)
-	(label "INTER_kmrkt_borden_2"
-		(at 250.19 168.91 180)
-		(effects
-			(font

Commit message: almost done, just silkscreen now
Parts:
- removed TP6: TestPoint, TestPoint:TestPoint_Pad_D2.0mm, symbol Connector:TestPoint
Connections:
- net IO10: now also TP7.1
- net IO1_SW: no longer TP7.1
Changed lines of the file:
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@@
 	(wire
 		(pts
-			(xy 349.25 280.67) (xy 355.6 280.67)
-		)
-		(stroke
-			(width 0)
-			(type default)
-		)
-	)
-	(wire
-		(pts
 			(xy 115.57 261.62) (xy 120.65 261.62)
 		)
@@
 		)
 	)
-	(label "IO1_SW"
+	(label "IO10"
 		(at 353.06 284.48 0)
 		(effects
@@
 		)
 	)
-	(label "IO0_SW"
-		(at 353.06 280.67 0)
-		(effects
-			(font
-				(size 1.27 1.27)
-			)
-			(justify left bottom)
-		)
-	)
 	(label "INTER_block_fairway_2"
 		(at 520.7 45.72 90)
@@
 					(unit 1)
 				)
-			)
-		)
-	)
-	(symbol
-		(lib_id "Connector:TestPoint")
-		(at 349.25 280.67 90)
-		(unit 1)
-		(exclude_from_sim no)
-		(in_bom yes)
-		(on_board yes)
-		(dnp no)
-		(property "Reference" "TP6"
-			(at 342.138 280.67 90)
-			(effects
-				(font
-					(size 1.27 1.27)
-				)
-			)
-		)
-		(property "Value" "TestPoint"
-			(at 334.518 280.67 90)
-			(effects
-				(font
-					(size 1.27 1.27)
-				)
-			)
-		)
-		(property "Footprint" "TestPoint:TestPoint_Pad_D2.0mm"
-			(at 349.25 275.59 0)
-			(effects
-				(font
-					(size 1.27 1.27)
-				)
-				(hide yes)
-			)
-		)
-		(property "Datasheet" "~"
-			(at 349.25 275.59 0)
-			(effects
-				(font
-					(size 1.27 1.27)
-				)
-				(hide yes)
-			)
-		)
-		(property "Description" "test point"
-			(at 349.25 280.67 0)
-			(effects
-				(font
-					(size 1.27 1.27)
-				)
-				(hide yes)
-			)
-		)
-		(pin "1"
-		)
-		(instances
-			(project "where_is_my_ion"
-				(path "/1b7d39dc-ea72-40bd-b392-fed3f2ced69f"
-					(reference "TP6")
-					(unit 1)
-				)
